Commit message: Add humanoid walking functionality and related components
- Implemented a new walking node (`humanoid_walk`) that handles footstep planning, CoM control, and inverse kinematics for humanoid robots.
- Enhanced the existing `humanoid_walking` node with inverse kinematics testing capabilities.
- Created a launch file (`walk.launch.py`) to facilitate the launching of the walking node with configurable parameters.
- Updated package dependencies in `package.xml` to include `humanoid_description` and `humanoid_interfaces`.
- Added configuration files and launch files to the package setup.
- Introduced unit tests for gait planning and walking patterns in `test/test_gait.py`.
- Modified URDF files to support floating base functionality for simulation.
- Defined a new action interface (`Walk.action`) for controlling the walking behavior of the humanoid robot.

File: src/humanoid_description/urdf/humanoid.xacro (robot description, xacro)
@@ -8,4 +8,14 @@
   <xacro:include filename="$(find humanoid_description)/urdf/transmissions/leg_transmissions_macro.xacro"/>
   <xacro:include filename="$(find humanoid_description)/urdf/ros2_control.xacro"/>
+  <!-- floating:=true pins the base in the air (for inspecting motions without falling) -->
+  <xacro:arg name="floating" default="false"/>
+  <xacro:if value="$(arg floating)">
+    <link name="world" />
+    <joint name="world_to_base" type="fixed">
+      <origin xyz="0 0 0" rpy="0 0 0" />
+      <parent link="world" />
+      <child link="base" />
+    </joint>
+  </xacro:if>
   <link name="base" />
   <joint name="base_to_torso" type="fixed">

File: src/humanoid_description/urdf/properties.xacro (robot description, xacro)
@@ -9,6 +9,6 @@
   <xacro:property name="shin_radius" value="0.06"/>
   <xacro:property name="shin_length" value="0.4"/>
-  <xacro:property name="foot_x" value="0.15"/>
-  <xacro:property name="foot_y" value="0.3"/>
+  <xacro:property name="foot_x" value="0.20"/>
+  <xacro:property name="foot_y" value="0.34"/>
   <xacro:property name="foot_z" value="0.05"/>
   <!-- Link mass properties -->

Commit message: Add step_n service and update humanoid walking functionality
- Introduced `/humanoid_walking/step_n` service for executing multiple alternating steps.
- Updated README with new service usage instructions.
- Adjusted timer interval in `humanoid_startup.py` for improved performance.
- Modified controller gains and properties in configuration files for better control.
- Updated physics engine settings in world configuration for enhanced simulation.
- Added `StepN.srv` for service interface and updated package description.

File: src/humanoid_description/urdf/humanoid.xacro (robot description, xacro)
@@ -33,14 +33,18 @@
   <xacro:humanoid_ros2_control/>
   <gazebo reference="left_foot_link">
-    <mu1>2.5</mu1>
-    <mu2>2.5</mu2>
-    <kp>500000.0</kp>
-    <kd>10.0</kd>
+    <mu1>1</mu1>
+    <mu2>1</mu2>
+    <kp>2000000.0</kp>
+    <kd>100.0</kd>
+    <min_depth>0.001</min_depth>
+    <max_vel>0.01</max_vel>
   </gazebo>
   <gazebo reference="right_foot_link">
-    <mu1>2.5</mu1>
-    <mu2>2.5</mu2>
-    <kp>500000.0</kp>
-    <kd>10.0</kd>
+    <mu1>1</mu1>
+    <mu2>1</mu2>
+    <kp>2000000.0</kp>
+    <kd>100.0</kd>
+    <min_depth>0.001</min_depth>
+    <max_vel>0.01</max_vel>
   </gazebo>
   <gazebo>

File: src/humanoid_description/urdf/properties.xacro (robot description, xacro)
@@ -13,5 +13,5 @@
   <xacro:property name="foot_z" value="0.05"/>
   <!-- Link mass properties -->
-  <xacro:property name="torso_mass" value="20.0"/>
+  <xacro:property name="torso_mass" value="12.0"/>
   <xacro:property name="hip_yaw_mass" value="0.1"/>
   <xacro:property name="hip_pitch_mass" value="0.1"/>
@@ -45,4 +45,4 @@
   <xacro:property name="ankle_pitch_limit_effort" value="120"/>
   <xacro:property name="ankle_roll_limit_effort" value="120"/>
-  <xacro:property name="leg_joint_limit_velocity" value="5.0"/>
+  <xacro:property name="leg_joint_limit_velocity" value="15.0"/>
 </robot>

Commit message: Add balance state message and related functionality
- Introduced a new message type `BalanceState` in `humanoid_interfaces` to publish the balance stabilizer state of the humanoid walk.
- Updated `CMakeLists.txt` and `package.xml` to include dependencies for the new message.
- Enhanced the `package.xml` of `humanoid_control` to include additional dependencies such as `control_msgs` and `nav_msgs`.
- Added new executables `gait_monitor` and `gait_check` in `setup.py`.
- Created a new test file `test_balance.py` to validate the functionality of the balance controller and state estimator.
- Added tests for support polygon calculations in `test_support_polygon.py`.
- Updated Gazebo parameters in `gazebo_params.yaml` for improved simulation performance.
- Modified the URDF files to include ankle force/torque sensors and adjusted joint limits for ankle roll.
- Updated the launch file to include the new Gazebo parameters.

File: src/humanoid_description/urdf/humanoid.xacro (robot description, xacro)
@@ -62,3 +62,27 @@
     </plugin>
   </gazebo>
+  <gazebo reference="left_ankle_pitch">
+    <provideFeedback>true</provideFeedback>
+  </gazebo>
+  <gazebo reference="right_ankle_pitch">
+    <provideFeedback>true</provideFeedback>
+  </gazebo>
+  <!-- Ankle force/torque sensors. They publish the ankle_pitch joint wrench in the
+       foot_link frame (ankle), measured from child (foot) to parent. -->
+  <gazebo>
+    <plugin name="left_foot_ft" filename="libgazebo_ros_ft_sensor.so">
+      <ros>
+        <remapping>wrench:=left_foot_ft</remapping>
+      </ros>
+      <joint_name>left_ankle_pitch</joint_name>
+      <update_rate>500.0</update_rate>
+    </plugin>
+    <plugin name="right_foot_ft" filename="libgazebo_ros_ft_sensor.so">
+      <ros>
+        <remapping>wrench:=right_foot_ft</remapping>
+      </ros>
+      <joint_name>right_ankle_pitch</joint_name>
+      <update_rate>500.0</update_rate>
+    </plugin>
+  </gazebo>
 </robot>

File: src/humanoid_description/urdf/properties.xacro (robot description, xacro)
@@ -37,6 +37,6 @@
   <xacro:property name="ankle_pitch_limit_lower" value="-0.5"/>
   <xacro:property name="ankle_pitch_limit_upper" value="0.8"/>
-  <xacro:property name="ankle_roll_limit_lower" value="-0.3"/>
-  <xacro:property name="ankle_roll_limit_upper" value="0.3"/>
+  <xacro:property name="ankle_roll_limit_lower" value="-0.4"/>
+  <xacro:property name="ankle_roll_limit_upper" value="0.4"/>
   <xacro:property name="hip_yaw_limit_effort" value="200"/>
   <xacro:property name="hip_roll_limit_effort" value="200"/>
